File: GuitarPedalBasic.kicad_pcb (KiCad board)
At the start: 2 copper layers, 49 x 40 mm, 21 parts, among them J1 INPUT, J2 OUTPUT, U1 TL082

Commit message: Without Tracks
Routing:
- net Net-(D1-K): track 0.00 -> 46.0 mm
- net Net-(D1-A): track 0.00 -> 45.3 mm, vias 0 -> 2
- net /9V: track 0.00 -> 37.0 mm, vias 0 -> 2
- net Net-(RV2-Pad3): track 0.00 -> 18.5 mm
- net Net-(J2-Pin_2): track 0.00 -> 16.6 mm
- net /4.5V: track 0.00 -> 15.2 mm, vias 0 -> 2
- net Net-(C7-Pad2): track 0.00 -> 11.3 mm
- net Net-(C6-Pad2): track 0.00 -> 10.9 mm
- net Net-(J1-Pin_2): track 0.00 -> 6.22 mm
- net Net-(R1-Pad1): track 0.00 -> 6.19 mm
- net Net-(C5-Pad1): track 0.00 -> 3.71 mm
- net Net-(C3-Pad1): track 0.00 -> 2.01 mm
