File: GuitarPedalBasic/GuitarPedalBasic.kicad_pcb (KiCad board)
At the start: 2 copper layers, 49 x 40 mm, 21 parts, among them J1 INPUT, J2 OUTPUT, U1 TL082

Commit message: PCB With SilkScreen Text
Parts:
- moved R3 10.6 mm to (32.9, 25.2)
- moved C4 10.6 mm to (36.8, 28.2)
- moved C5 10.6 mm to (39.5, 35.1)
- moved U1 10.6 mm to (43.1, 29.7)
- moved BT1 10.6 mm to (19.2, 21.0)
- moved C1 10.6 mm to (27.8, 18.8)
- moved C3 10.6 mm to (30.2, 27.5)
- moved C7 10.6 mm to (30.8, 35.6)
- moved J1 10.6 mm to (19.2, 31.0)
- moved R1 10.6 mm to (25.8, 24.3)
- moved R2 10.6 mm to (29.2, 24.3)
- moved RV1 10.6 mm to (20.0, 38.5)
- moved C2 10.6 mm to (34.1, 18.8)
- moved C6 10.6 mm to (46.0, 35.1)
- moved D1 10.6 mm to (43.1, 24.0)
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Other:
- board text added: "AUDIO IN"
- board text added: "AUDIO OUT"
- board text added: "GAIN"
- board text added: "GND"
- board text added: "TONE"
- board text added: "VCC"
- board text added: "VOLUME"

Commit message: Simulations added
Routing:
- net GND: vias 0 -> 4
